File: pcb/the-matrix.kicad_sch (KiCad schematic)
At the start: 81 parts, among them J1 DNP, J2 DNP, J3 Conn_02x20_Odd_Even, J4 Conn_02x20_Odd_Even, J5 Conn_02x20_Odd_Even, J6 Conn_02x20_Odd_Even, Q1 Q_PMOS_GDS, Q10 Q_PMOS_GDS, Q11 Q_PMOS_GDS, Q12 Q_PMOS_GDS, Q13 Q_PMOS_GDS, Q14 Q_PMOS_GDS, Q15 Q_PMOS_GDS, Q16 Q_PMOS_GDS, Q17 Q_PMOS_GDS, Q18 Q_PMOS_GDS, Q19 Q_PMOS_GDS, Q2 Q_PMOS_GDS, Q20 Q_PMOS_GDS, Q21 Q_PMOS_GDS, Q22 Q_PMOS_GDS, Q23 Q_PMOS_GDS, Q24 Q_PMOS_GDS, Q25 Q_PMOS_GDS, Q26 Q_PMOS_GDS, Q27 Q_PMOS_GDS, Q28 Q_PMOS_GDS, Q29 Q_PMOS_GDS, Q3 Q_PMOS_GDS, Q30 Q_PMOS_GDS, Q31 Q_PMOS_GDS, Q32 Q_PMOS_GDS, Q33 Q_PMOS_GDS, Q34 Q_PMOS_GDS, Q35 Q_PMOS_GDS, Q36 Q_PMOS_GDS, Q37 Q_PMOS_GDS, Q38 Q_PMOS_GDS, Q39 Q_PMOS_GDS, Q4 Q_PMOS_GDS, Q40 Q_PMOS_GDS, Q5 Q_PMOS_GDS, Q6 Q_PMOS_GDS, Q7 Q_PMOS_GDS, Q8 Q_PMOS_GDS, Q9 Q_PMOS_GDS, U1 74HC595, U10 TPIC6B595N, U2 74HC595, U3 74HC595, U4 74HC595, U5 74HC595, U6 TPIC6B595N, U7 TPIC6B595N, U8 TPIC6B595N, U9 TPIC6B595N

Commit message: an amount of progress on routing
Parts:
- J1, J2: now not fitted
- Q1, Q10, Q11, Q12, Q13, Q14, Q15, Q16, Q17, Q18, Q19, Q2, Q20, Q21, Q22, Q23, Q24, Q25, Q26, Q27, Q28, Q29, Q3, Q30, Q31, Q32, Q33, Q34, Q35, Q36, Q37, Q38, Q39, Q4, Q40, Q5, Q6, Q7, Q8, Q9: footprint Package_TO_SOT_THT:TO-251-3_Vertical -> TO-251-ThinPads:TO-251-3_Vertical_ThinPads
Changed lines of the file:
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@@
 			)
 		)
-		(property "Footprint" "Package_TO_SOT_THT:TO-251-3_Vertical"
+		(property "Footprint" "TO-251-ThinPads:TO-251-3_Vertical_ThinPads"
 			(at 341.63 66.04 0)
 			(effects
@@
 			)
 		)
-		(property "Footprint" "Package_TO_SOT_THT:TO-251-3_Vertical"
+		(property "Footprint" "TO-251-ThinPads:TO-251-3_Vertical_ThinPads"
 			(at 463.55 66.04 0)
 			(effects
@@
 			)
 		)
-		(property "Footprint" "Package_TO_SOT_THT:TO-251-3_Vertical"
+		(property "Footprint" "TO-251-ThinPads:TO-251-3_Vertical_ThinPads"
 			(at 326.39 73.66 0)
 			(effects
@@
 			)
 		)
-		(property "Footprint" "Package_TO_SOT_THT:TO-251-3_Vertical"
+		(property "Footprint" "TO-251-ThinPads:TO-251-3_Vertical_ThinPads"
 			(at 570.23 73.66 0)
 			(effects
@@
 			)
 		)
-		(property "Footprint" "Package_TO_SOT_THT:TO-251-3_Vertical"
+		(property "Footprint" "TO-251-ThinPads:TO-251-3_Vertical_ThinPads"
 			(at 468.63 73.66 0)
 			(effects
@@
 			)
 		)
-		(property "Footprint" "Package_TO_SOT_THT:TO-251-3_Vertical"
+		(property "Footprint" "TO-251-ThinPads:TO-251-3_Vertical_ThinPads"
 			(at 336.55 58.42 0)
 			(effects
@@
 			)
 		)
-		(property "Footprint" "Package_TO_SOT_THT:TO-251-3_Vertical"
+		(property "Footprint" "TO-251-ThinPads:TO-251-3_Vertical_ThinPads"
 			(at 529.59 73.66 0)
 			(effects
@@
 			)
 		)
-		(property "Footprint" "Package_TO_SOT_THT:TO-251-3_Vertical"
+		(property "Footprint" "TO-251-ThinPads:TO-251-3_Vertical_ThinPads"
 			(at 560.07 58.42 0)
 			(effects
@@
 			)
 		)
-		(property "Footprint" "Package_TO_SOT_THT:TO-251-3_Vertical"
+		(property "Footprint" "TO-251-ThinPads:TO-251-3_Vertical_ThinPads"
 			(at 590.55 73.66 0)
 			(effects
@@
 			)
 		)
-		(property "Footprint" "Package_TO_SOT_THT:TO-251-3_Vertical"
+		(property "Footprint" "TO-251-ThinPads:TO-251-3_Vertical_ThinPads"
 			(at 473.71 81.28 0)
 			(effects
@@
 			)
 		)
-		(property "Footprint" "Package_TO_SOT_THT:TO-251-3_Vertical"
+		(property "Footprint" "TO-251-ThinPads:TO-251-3_Vertical_ThinPads"
 			(at 346.71 73.66 0)
 			(effects
@@
 			)
 		)
-		(property "Footprint" "Package_TO_SOT_THT:TO-251-3_Vertical"
+		(property "Footprint" "TO-251-ThinPads:TO-251-3_Vertical_ThinPads"
 			(at 519.43 58.42 0)
 			(effects
@@
 			)
 		)
-		(property "Footprint" "Package_TO_SOT_THT:TO-251-3_Vertical"
+		(property "Footprint" "TO-251-ThinPads:TO-251-3_Vertical_ThinPads"
 			(at 397.51 58.42 0)
 			(effects
@@
 			)
 		)
-		(property "Footprint" "Package_TO_SOT_THT:TO-251-3_Vertical"
+		(property "Footprint" "TO-251-ThinPads:TO-251-3_Vertical_ThinPads"
 			(at 351.79 81.28 0)
 			(effects
@@
 			)
 		)
-		(property "Footprint" "Package_TO_SOT_THT:TO-251-3_Vertical"
+		(property "Footprint" "TO-251-ThinPads:TO-251-3_Vertical_ThinPads"
 			(at 407.67 73.66 0)
 			(effects
@@
 			)
 		)
-		(property "Footprint" "Package_TO_SOT_THT:TO-251-3_Vertical"
+		(property "Footprint" "TO-251-ThinPads:TO-251-3_Vertical_ThinPads"
 			(at 565.15 66.04 0)
 			(effects
@@
 			)
 		)
-		(property "Footprint" "Package_TO_SOT_THT:TO-251-3_Vertical"
+		(property "Footprint" "TO-251-ThinPads:TO-251-3_Vertical_ThinPads"
 			(at 316.23 58.42 0)
 			(effects
@@
 			)
 		)
-		(property "Footprint" "Package_TO_SOT_THT:TO-251-3_Vertical"
+		(property "Footprint" "TO-251-ThinPads:TO-251-3_Vertical_ThinPads"
 			(at 534.67 81.28 0)
 			(effects
@@
 			)
 		)
-		(property "Footprint" "Package_TO_SOT_THT:TO-251-3_Vertical"
+		(property "Footprint" "TO-251-ThinPads:TO-251-3_Vertical_ThinPads"
 			(at 382.27 66.04 0)
 			(effects
@@
 			)
 		)
-		(property "Footprint" "Package_TO_SOT_THT:TO-251-3_Vertical"
+		(property "Footprint" "TO-251-ThinPads:TO-251-3_Vertical_ThinPads"
 			(at 509.27 73.66 0)
 			(effects
@@
 			)
 		)
-		(property "Footprint" "Package_TO_SOT_THT:TO-251-3_Vertical"
+		(property "Footprint" "TO-251-ThinPads:TO-251-3_Vertical_ThinPads"
 			(at 402.59 66.04 0)
 			(effects
@@
 			)
 		)
-		(property "Footprint" "Package_TO_SOT_THT:TO-251-3_Vertical"
+		(property "Footprint" "TO-251-ThinPads:TO-251-3_Vertical_ThinPads"
 			(at 392.43 81.28 0)
 			(effects
@@
 			)
 		)
-		(property "Footprint" "Package_TO_SOT_THT:TO-251-3_Vertical"
+		(property "Footprint" "TO-251-ThinPads:TO-251-3_Vertical_ThinPads"
 			(at 595.63 81.28 0)
 			(effects
@@
 			)
 		)
-		(property "Footprint" "Package_TO_SOT_THT:TO-251-3_Vertical"
+		(property "Footprint" "TO-251-ThinPads:TO-251-3_Vertical_ThinPads"
 			(at 377.19 58.42 0)
 			(effects
@@
 			)
 		)
-		(property "Footprint" "Package_TO_SOT_THT:TO-251-3_Vertical"
+		(property "Footprint" "TO-251-ThinPads:TO-251-3_Vertical_ThinPads"
 			(at 585.47 66.04 0)
 			(effects
@@
 		(in_bom yes)
 		(on_board yes)
-		(dnp no)
+		(dnp yes)
 		(fields_autoplaced yes)
 		(property "Reference" "J1"
@@
 			)
 		)
-		(property "Footprint" "Package_TO_SOT_THT:TO-251-3_Vertical"
+		(property "Footprint" "TO-251-ThinPads:TO-251-3_Vertical_ThinPads"
 			(at 499.11 58.42 0)
 			(effects
@@
 			)
 		)
-		(property "Footprint" "Package_TO_SOT_THT:TO-251-3_Vertical"
+		(property "Footprint" "TO-251-ThinPads:TO-251-3_Vertical_ThinPads"
 			(at 387.35 73.66 0)
 			(effects
@@
 			)
 		)
-		(property "Footprint" "Package_TO_SOT_THT:TO-251-3_Vertical"
+		(property "Footprint" "TO-251-ThinPads:TO-251-3_Vertical_ThinPads"
 			(at 580.39 58.42 0)
 			(effects
@@
 			)
 		)
-		(property "Footprint" "Package_TO_SOT_THT:TO-251-3_Vertical"
+		(property "Footprint" "TO-251-ThinPads:TO-251-3_Vertical_ThinPads"
 			(at 321.31 66.04 0)
 			(effects
@@
 		(in_bom yes)
 		(on_board yes)
-		(dnp no)
+		(dnp yes)
 		(fields_autoplaced yes)
 		(property "Reference" "J2"
@@
 			)
 		)
-		(property "Footprint" "Package_TO_SOT_THT:TO-251-3_Vertical"
+		(property "Footprint" "TO-251-ThinPads:TO-251-3_Vertical_ThinPads"
 			(at 524.51 66.04 0)
 			(effects
@@
 			)
 		)
-		(property "Footprint" "Package_TO_SOT_THT:TO-251-3_Vertical"
+		(property "Footprint" "TO-251-ThinPads:TO-251-3_Vertical_ThinPads"
 			(at 412.75 81.28 0)
 			(effects
@@
 			)
 		)
-		(property "Footprint" "Package_TO_SOT_THT:TO-251-3_Vertical"
+		(property "Footprint" "TO-251-ThinPads:TO-251-3_Vertical_ThinPads"
 			(at 504.19 66.04 0)
 			(effects
@@
 			)
 		)
-		(property "Footprint" "Package_TO_SOT_THT:TO-251-3_Vertical"
+		(property "Footprint" "TO-251-ThinPads:TO-251-3_Vertical_ThinPads"
 			(at 443.23 66.04 0)
 			(effects
@@
 			)
 		)
-		(property "Footprint" "Package_TO_SOT_THT:TO-251-3_Vertical"
+		(property "Footprint" "TO-251-ThinPads:TO-251-3_Vertical_ThinPads"
 			(at 448.31 73.66 0)
 			(effects
@@
 			)
 		)
-		(property "Footprint" "Package_TO_SOT_THT:TO-251-3_Vertical"
+		(property "Footprint" "TO-251-ThinPads:TO-251-3_Vertical_ThinPads"
 			(at 453.39 81.28 0)
 			(effects
@@
 			)
 		)
-		(property "Footprint" "Package_TO_SOT_THT:TO-251-3_Vertical"
+		(property "Footprint" "TO-251-ThinPads:TO-251-3_Vertical_ThinPads"
 			(at 514.35 81.28 0)
 			(effects
@@
 			)
 		)
-		(property "Footprint" "Package_TO_SOT_THT:TO-251-3_Vertical"
+		(property "Footprint" "TO-251-ThinPads:TO-251-3_Vertical_ThinPads"
 			(at 331.47 81.28 0)
 			(effects
@@
 			)
 		)
-		(property "Footprint" "Package_TO_SOT_THT:TO-251-3_Vertical"
+		(property "Footprint" "TO-251-ThinPads:TO-251-3_Vertical_ThinPads"
 			(at 575.31 81.28 0)
 			(effects
@@
 			)
 		)
-		(property "Footprint" "Package_TO_SOT_THT:TO-251-3_Vertical"
+		(property "Footprint" "TO-251-ThinPads:TO-251-3_Vertical_ThinPads"
 			(at 458.47 58.42 0)
 			(effects
@@
 			)
 		)
-		(property "Footprint" "Package_TO_SOT_THT:TO-251-3_Vertical"
+		(property "Footprint" "TO-251-ThinPads:TO-251-3_Vertical_ThinPads"
 			(at 438.15 58.42 0)
 			(effects

Commit message: route the matrix
Connections:
- net COLA0: now also J3.39 (Pin_39), J6.40 (Pin_40); no longer J3.1 (Pin_1), J6.2 (Pin_2)
- net COLA1: now also J3.40 (Pin_40), J6.39 (Pin_39); no longer J3.2 (Pin_2), J6.1 (Pin_1)
- net COLA10: now also J3.29 (Pin_29), J6.30 (Pin_30); no longer J3.11 (Pin_11), J6.12 (Pin_12)
- net COLA11: now also J3.30 (Pin_30), J6.29 (Pin_29); no longer J3.12 (Pin_12), J6.11 (Pin_11)
- net COLA12: now also J3.27 (Pin_27), J6.28 (Pin_28); no longer J3.13 (Pin_13), J6.14 (Pin_14)
- net COLA13: now also J3.28 (Pin_28), J6.27 (Pin_27); no longer J3.14 (Pin_14), J6.13 (Pin_13)
- net COLA14: now also J3.25 (Pin_25), J6.26 (Pin_26); no longer J3.15 (Pin_15), J6.16 (Pin_16)
- net COLA15: now also J3.26 (Pin_26), J6.25 (Pin_25); no longer J3.16 (Pin_16), J6.15 (Pin_15)
- net COLA16: now also J3.23 (Pin_23), J6.24 (Pin_24); no longer J3.17 (Pin_17), J6.18 (Pin_18)
- net COLA17: now also J3.24 (Pin_24), J6.23 (Pin_23); no longer J3.18 (Pin_18), J6.17 (Pin_17)
- net COLA18: now also J3.21 (Pin_21), J6.22 (Pin_22); no longer J3.19 (Pin_19), J6.20 (Pin_20)
- net COLA19: now also J3.22 (Pin_22), J6.21 (Pin_21); no longer J3.20 (Pin_20), J6.19 (Pin_19)
- net COLA2: now also J3.37 (Pin_37), J6.38 (Pin_38); no longer J3.3 (Pin_3), J6.4 (Pin_4)
- net COLA20: now also J3.19 (Pin_19), J6.20 (Pin_20); no longer J3.21 (Pin_21), J6.22 (Pin_22)
- net COLA21: now also J3.20 (Pin_20), J6.19 (Pin_19); no longer J3.22 (Pin_22), J6.21 (Pin_21)
- net COLA22: now also J3.17 (Pin_17), J6.18 (Pin_18); no longer J3.23 (Pin_23), J6.24 (Pin_24)
- net COLA23: now also J3.18 (Pin_18), J6.17 (Pin_17); no longer J3.24 (Pin_24), J6.23 (Pin_23)
- net COLA24: now also J3.15 (Pin_15), J6.16 (Pin_16); no longer J3.25 (Pin_25), J6.26 (Pin_26)
- net COLA25: now also J3.16 (Pin_16), J6.15 (Pin_15); no longer J3.26 (Pin_26), J6.25 (Pin_25)
- net COLA26: now also J3.13 (Pin_13), J6.14 (Pin_14); no longer J3.27 (Pin_27), J6.28 (Pin_28)
- net COLA27: now also J3.14 (Pin_14), J6.13 (Pin_13); no longer J3.28 (Pin_28), J6.27 (Pin_27)
- net COLA28: now also J3.11 (Pin_11), J6.12 (Pin_12); no longer J3.29 (Pin_29), J6.30 (Pin_30)
- net COLA29: now also J3.12 (Pin_12), J6.11 (Pin_11); no longer J3.30 (Pin_30), J6.29 (Pin_29)
- net COLA3: now also J3.38 (Pin_38), J6.37 (Pin_37); no longer J3.4 (Pin_4), J6.3 (Pin_3)
- net COLA30: now also J3.9 (Pin_9), J6.10 (Pin_10); no longer J3.31 (Pin_31), J6.32 (Pin_32)
- net COLA31: now also J3.10 (Pin_10), J6.9 (Pin_9); no longer J3.32 (Pin_32), J6.31 (Pin_31)
- net COLA32: now also J3.7 (Pin_7), J6.8 (Pin_8); no longer J3.33 (Pin_33), J6.34 (Pin_34)
- net COLA33: now also J3.8 (Pin_8), J6.7 (Pin_7); no longer J3.34 (Pin_34), J6.33 (Pin_33)
- net COLA34: now also J3.5 (Pin_5), J6.6 (Pin_6); no longer J3.35 (Pin_35), J6.36 (Pin_36)
- net COLA35: now also J3.6 (Pin_6), J6.5 (Pin_5); no longer J3.36 (Pin_36), J6.35 (Pin_35)
- net COLA36: now also J3.3 (Pin_3), J6.4 (Pin_4); no longer J3.37 (Pin_37), J6.38 (Pin_38)
- net COLA37: now also J3.4 (Pin_4), J6.3 (Pin_3); no longer J3.38 (Pin_38), J6.37 (Pin_37)
- net COLA38: now also J3.1 (Pin_1), J6.2 (Pin_2); no longer J3.39 (Pin_39), J6.40 (Pin_40)
- net COLA39: now also J3.2 (Pin_2), J6.1 (Pin_1); no longer J3.40 (Pin_40), J6.39 (Pin_39)
- net COLA4: now also J3.35 (Pin_35), J6.36 (Pin_36); no longer J3.5 (Pin_5), J6.6 (Pin_6)
- net COLA5: now also J3.36 (Pin_36), J6.35 (Pin_35); no longer J3.6 (Pin_6), J6.5 (Pin_5)
- net COLA6: now also J3.33 (Pin_33), J6.34 (Pin_34); no longer J3.7 (Pin_7), J6.8 (Pin_8)
- net COLA7: now also J3.34 (Pin_34), J6.33 (Pin_33); no longer J3.8 (Pin_8), J6.7 (Pin_7)
- net COLA8: now also J3.31 (Pin_31), J6.32 (Pin_32); no longer J3.9 (Pin_9), J6.10 (Pin_10)
- net COLA9: now also J3.32 (Pin_32), J6.31 (Pin_31); no longer J3.10 (Pin_10), J6.9 (Pin_9)
Other:
- moved on the sheet: J3, J6
Changed lines of the file:
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@@
 	(symbol
 		(lib_id "Connector_Generic:Conn_02x20_Odd_Even")
-		(at 132.08 179.07 90)
-		(mirror x)
+		(at 134.62 179.07 270)
 		(unit 1)
 		(exclude_from_sim no)
@@
 		(dnp no)
 		(property "Reference" "J6"
-			(at 102.87 180.34 0)
+			(at 163.83 180.34 0)
 			(effects
 				(font
@@
 		)
 		(property "Value" "Conn_02x20_Odd_Even"
-			(at 105.41 180.34 0)
+			(at 161.29 180.34 0)
 			(effects
 				(font
@@
 		)
 		(property "Footprint" "Connector_PinSocket_2.54mm:PinSocket_2x20_P2.54mm_Horizontal"
-			(at 132.08 179.07 0)
+			(at 134.62 179.07 0)
 			(effects
 				(font
@@
 		)
 		(property "Datasheet" "~"
-			(at 132.08 179.07 0)
+			(at 134.62 179.07 0)
 			(effects
 				(font
@@
 		)
 		(property "Description" "Generic connector, double row, 02x20, odd/even pin numbering scheme (row 1 odd numbers, row 2 even numbers), script generated (kicad-library-utils/schlib/autogen/connector/)"
-			(at 132.08 179.07 0)
+			(at 134.62 179.07 0)
 			(effects
 				(font
@@
 	(symbol
 		(lib_id "Connector_Generic:Conn_02x20_Odd_Even")
-		(at 132.08 93.98 90)
-		(mirror x)
+		(at 134.62 93.98 270)
 		(unit 1)
 		(exclude_from_sim no)
@@
 		(on_board yes)
 		(dnp no)
-		(fields_autoplaced yes)
 		(property "Reference" "J3"
-			(at 102.87 95.25 0)
+			(at 163.83 95.25 0)
 			(effects
 				(font
@@
 		)
 		(property "Value" "Conn_02x20_Odd_Even"
-			(at 105.41 95.25 0)
+			(at 161.29 95.25 0)
 			(effects
 				(font
@@
 		)
 		(property "Footprint" "Connector_PinHeader_2.54mm:PinHeader_2x20_P2.54mm_Horizontal"
-			(at 132.08 93.98 0)
+			(at 134.62 93.98 0)
 			(effects
 				(font
@@
 		)
 		(property "Datasheet" "~"
-			(at 132.08 93.98 0)
+			(at 134.62 93.98 0)
 			(effects
 				(font
@@
 		)
 		(property "Description" "Generic connector, double row, 02x20, odd/even pin numbering scheme (row 1 odd numbers, row 2 even numbers), script generated (kicad-library-utils/schlib/autogen/connector/)"
-			(at 132.08 93.98 0)
-			(effects
-				(font
+			(at 134.62 93.98 0)
+			(effects
+				(font
