File: pcb/the-matrix.kicad_pcb (KiCad board)
At the start: 4 copper layers, 102 x 102 mm, 81 parts, among them J1 DNP, J2 DNP, J3 Conn_02x20_Odd_Even, J4 Conn_02x20_Odd_Even, J5 Conn_02x20_Odd_Even, J6 Conn_02x20_Odd_Even, Q1 Q_PMOS_GDS, Q10 Q_PMOS_GDS, Q11 Q_PMOS_GDS, Q12 Q_PMOS_GDS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

Commit message: before resistor silkscreen reexport
Other:
- board text added: "ROW CONTROL"
